File: analog-keeb-proto.kicad_pcb (KiCad board)
At the start: 2 copper layers, 150 parts, among them J1 USB_C_Receptacle_USB2.0_16P, J3 Conn_01x05, SW1 SW_Push, SW2 SW_Push, U1 RP2040, U2 XC6206PxxxMR, U3 SRV05-4, U30 CD74HC4067SM, U4 W25Q128JVS, Y1 ABM8-272-T3

Commit message: trol
Parts:
- C1, C10, C100, C101, C102, C103, C104, C105, C11, C12, C13, C14, C15, C16, C17, C18, C19, C2, C20, C21, C22, C23, C24, C25, C26, C27, C28, C29, C3, C32, C33, C34, C35, C36, C37, C38, C39, C4, C42, C43, C44, C45, C46, C47, C48, C49, C5, C52, C53, C54, C55, C56, C57, C58, C59, C6, C7, C8, C86, C87, C88, C89, C9, C90, C91, C92, C93, C94, C95, C96, C97, C98, C99, D1, D10, D11, D12, D13, D14, D15, D16, D17, D18, D19, D2, D20, D21, D22, D23, D24, D25, D3, D4, D5, D6, D7, D8, D9, F1, J1, J3, R1, R2, R3, R4, R5, R6, R7, R8, R9, SW1, SW2, U1, U10, U11, U12, U13, U14, U15, U16, U17, U18, U19, U2, U20, U21, U22, U23, U24, U25, U26, U27, U28, U29, U3, U30, U31, U32, U33, U34, U35, U36, U37, U4, U5, U6, U7, U8, U9, Y1: moved to B.Cu
- moved C1 183.8 mm to (252.1, 114.5), turned to 180 degrees
- moved C10 183.8 mm to (252.1, 129.3), turned to 180 degrees
- moved C11 183.8 mm to (252.1, 131.0), turned to 180 degrees
- moved C2 183.8 mm to (252.1, 116.1), turned to 180 degrees
- moved C3 183.8 mm to (252.1, 117.8), turned to 180 degrees
- moved C4 183.8 mm to (252.1, 119.4), turned to 180 degrees
- moved C5 183.8 mm to (252.1, 121.1), turned to 180 degrees
- moved C6 183.8 mm to (252.1, 122.7), turned to 180 degrees
- moved C7 183.8 mm to (252.1, 124.4), turned to 180 degrees
- moved C8 183.8 mm to (252.1, 126.0), turned to 180 degrees
- moved C9 183.8 mm to (252.1, 127.7), turned to 180 degrees
- moved C12 179.3 mm to (249.9, 114.5), turned to 180 degrees
- moved C13 179.3 mm to (249.9, 116.1), turned to 180 degrees
- moved C14 179.3 mm to (249.9, 117.8), turned to 180 degrees
- moved C15 179.3 mm to (249.9, 119.4), turned to 180 degrees
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Connections:
- U3 pad 1: D+ -> unconnected-(U3-IO1-Pad1)
- U3 pad 4: unconnected-(U3-IO3-Pad4) -> D+
- U30 pad 24: unconnected-(U30-VCC-Pad24) -> +5V
Routing:
- net GND: track 0.00 -> 49.1 mm, vias 0 -> 3
- net VBUS: track 0.00 -> 13.5 mm
- net D-: track 0.00 -> 12.2 mm
- net D+: track 0.00 -> 8.70 mm
- net Net-(U1-USB_DM): track 0.00 -> 7.64 mm
- net Net-(U1-USB_DP): track 0.00 -> 7.55 mm
- net +5V: track 0.00 -> 5.74 mm
- net Net-(J1-CC2): track 0.00 -> 4.54 mm
- net Net-(J1-CC1): track 0.00 -> 3.79 mm
- net +3V3: track 0.00 -> 2.24 mm
