File: analog-keeb-proto.kicad_sch (KiCad schematic)
At the start: 142 parts, among them J1 USB_C_Receptacle_USB2.0_16P, SW1 SW_Push, SW2 SW_Push, U1 RP2040, U2 XC6206PxxxMR, U3 SRV05-4, U30 CD74HC4067SM, U38 CD74HC4067SM, U4 W25Q128JVS, Y1 ABMB-272-T3

Commit message: add footprints
Parts:
- removed D1, D2, D26, D3, D4: SK6812MINI, LED_SMD:LED_SK6812MINI_PLCC4_3.5x3.5mm_P1.75mm, symbol LED:SK6812MINI
- added C100, C101, C102, C103, C104, C105, C86, C87, C88, C89, C90, C91, C92, C93, C94, C95, C96, C97, C98, C99: 100nF, Capacitor_SMD:C_01005_0402Metric, symbol Device:C
- added D1, D10, D11, D12, D13, D14, D15, D16, D17, D18, D19, D2, D20, D21, D22, D23, D24, D25, D3, D4, D5, D6, D7, D8, D9: SK6805, LED_SMD:LED_SK6805_PLCC4_2.4x2.7mm_P1.3mm, symbol LED:SK6805
- added J2: Conn_01x04, Connector_JST:JST_SH_SM04B-SRSS-TB_1x04-1MP_P1.00mm_Horizontal, symbol Connector_Generic:Conn_01x04
- added J3: Conn_01x05, Connector_PinHeader_2.54mm:PinHeader_1x05_P2.54mm_Vertical, symbol Connector_Generic:Conn_01x05
- C1, C10, C11, C12, C14, C15, C16, C17, C18, C19, C2, C20, C21, C22, C23, C3, C4, C5, C6, C7, C8, C9: footprint (none) -> Capacitor_SMD:C_01005_0402Metric
- C13: value 1u -> 100n; footprint (none) -> Capacitor_SMD:C_01005_0402Metric
- C24, C26, C28, C30, C31, C32, C34, C36, C38, C40, C41, C42, C44, C46, C48, C52, C54, C56, C58, C62, C63, C64, C65, C70, C71, C72, C73, C78, C79, C80, C81: value 1nF -> 10pF; footprint (none) -> Capacitor_SMD:C_01005_0402Metric
- C25, C27, C29, C33, C35, C37, C39, C43, C45, C47, C49, C50, C51, C53, C55, C57, C59, C60, C61, C66, C67, C68, C69, C74, C75, C76, C77, C82, C83, C84, C85: value 10pF -> 1nF; footprint (none) -> Capacitor_SMD:C_01005_0402Metric
- F1: footprint (none) -> Fuse:Fuse_1206_3216Metric
- J1: footprint (none) -> Connector_USB:USB_C_Receptacle_HRO_TYPE-C-31-M-12
- R1, R2, R3, R4, R5, R6, R7, R8, R9: footprint (none) -> Resistor_SMD:R_0402_1005Metric
- SW1, SW2: footprint (none) -> Button_Switch_SMD:SW_SPST_TL3342
- U10, U11, U12, U13, U14, U15, U16, U17, U18, U19, U20, U21, U22, U23, U24, U25, U26, U27, U28, U29, U31, U32, U33, U34, U35, U36, U37, U5, U6, U7, U8, U9: footprint (none) -> analog-keeb:HX6659-SOT23
- Y1: value ABMB-272-T3 -> ABM8-272-T3; footprint (none) -> Crystal:Crystal_SMD_3225-4Pin_3.2x2.5mm
Connections:
- net +3V3: now also J3.2 (Pin_2)
- net +5V: now also C22.1, C25.1, C27.1, C29.1, C33.1, C35.1, C37.1, C39.1, C43.1, C45.1, C47.1, C49.1, C50.1, C51.1, C53.1, C55.1, C57.1, C59.1, C60.1, C61.1, C66.1, C67.1, C68.1, C69.1, C74.1, C75.1, C76.1, C77.1, C82.1, C83.1, C84.1, C85.1, U10.1 (VCC), U11.1 (VCC), U12.1 (VCC), U13.1 (VCC), U14.1 (VCC), U15.1 (VCC), U16.1 (VCC), U17.1 (VCC), U18.1 (VCC), U19.1 (VCC), U20.1 (VCC), U21.1 (VCC), U22.1 (VCC), U23.1 (VCC), U24.1 (VCC), U25.1 (VCC), U26.1 (VCC), U27.1 (VCC), U28.1 (VCC), U29.1 (VCC), U31.1 (VCC), U32.1 (VCC), U33.1 (VCC), U34.1 (VCC), U35.1 (VCC), U36.1 (VCC), U37.1 (VCC), U5.1 (VCC), U6.1 (VCC), U7.1 (VCC), U8.1 (VCC), U9.1 (VCC), C100.2, C101.2, C102.2, C103.2, C104.2, C105.2, C86.2, C87.2, C88.2, C89.2, C90.2, C91.2, C92.2, C93.2, C94.2, C95.2, C96.2, C97.2, C98.2, C99.2, D1.4 (VDD), D10.4 (VDD), D11.4 (VDD), D12.4 (VDD), D13.4 (VDD), D14.4 (VDD), D15.4 (VDD), D16.4 (VDD), D17.4 (VDD), D18.4 (VDD), D19.4 (VDD), D2.4 (VDD), D20.4 (VDD), D21.4 (VDD), D22.4 (VDD), D23.4 (VDD), D24.4 (VDD), D25.4 (VDD), D3.4 (VDD), D4.4 (VDD), D5.4 (VDD), D6.4 (VDD), D7.4 (VDD), D8.4 (VDD), D9.4 (VDD), J2.1 (Pin_1); no longer C22.2, C24.2, C26.2, C28.2, C30.2, C31.2, C32.2, C34.2, C36.2, C38.2, C40.2, C41.2, C42.2, C44.2, C46.2, C48.2, C52.2, C54.2, C56.2, C58.2, C62.2, C63.2, C64.2, C65.2, C70.2, C71.2, C72.2, C73.2, C78.2, C79.2, C80.2, C81.2, U10. (OUT), U11. (OUT), U12. (OUT), U13. (OUT), U14. (OUT), U15. (OUT), U16. (OUT), U17. (OUT), U18. (OUT), U19. (OUT), U20. (OUT), U21. (OUT), U22. (OUT), U23. (OUT), U24. (OUT), U25. (OUT), U26. (OUT), U27. (OUT), U28. (OUT), U29. (OUT), U31. (OUT), U32. (OUT), U33. (OUT), U34. (OUT), U35. (OUT), U36. (OUT), U37. (OUT), U5. (OUT), U6. (OUT), U7. (OUT), U8. (OUT), U9. (OUT)
- net D+: now also J2.3 (Pin_3)
- net D-: now also J2.2 (Pin_2)
- net GND: now also C22.2, C25.2, C27.2, C29.2, C33.2, C35.2, C37.2, C39.2, C43.2, C45.2, C47.2, C49.2, C50.2, C51.2, C53.2, C55.2, C57.2, C59.2, C60.2, C61.2, C66.2, C67.2, C68.2, C69.2, C74.2, C75.2, C76.2, C77.2, C82.2, C83.2, C84.2, C85.2, U10.3 (GND), U11.3 (GND), U12.3 (GND), U13.3 (GND), U14.3 (GND), U15.3 (GND), U16.3 (GND), U17.3 (GND), U18.3 (GND), U19.3 (GND), U20.3 (GND), U21.3 (GND), U22.3 (GND), U23.3 (GND), U24.3 (GND), U25.3 (GND), U26.3 (GND), U27.3 (GND), U28.3 (GND), U29.3 (GND), U31.3 (GND), U32.3 (GND), U33.3 (GND), U34.3 (GND), U35.3 (GND), U36.3 (GND), U37.3 (GND), U5.3 (GND), U6.3 (GND), U7.3 (GND), U8.3 (GND), U9.3 (GND), C100.1, C101.1, C102.1, C103.1, C104.1, C105.1, C86.1, C87.1, C88.1, C89.1, C90.1, C91.1, C92.1, C93.1, C94.1, C95.1, C96.1, C97.1, C98.1, C99.1, D1.2 (VSS), D10.2 (VSS), D11.2 (VSS), D12.2 (VSS), D13.2 (VSS), D14.2 (VSS), D15.2 (VSS), D16.2 (VSS), D17.2 (VSS), D18.2 (VSS), D19.2 (VSS), D2.2 (VSS), D20.2 (VSS), D21.2 (VSS), D22.2 (VSS), D23.2 (VSS), D24.2 (VSS), D25.2 (VSS), D3.2 (VSS), D4.2 (VSS), D5.2 (VSS), D6.2 (VSS), D7.2 (VSS), D8.2 (VSS), D9.2 (VSS), J2.4 (Pin_4), J3.3 (Pin_3); no longer C22.1, C25.1, C27.1, C29.1, C33.1, C35.1, C37.1, C39.1, C43.1, C45.1, C47.1, C49.1, C50.1, C51.1, C53.1, C55.1, C57.1, C59.1, C60.1, C61.1, C66.1, C67.1, C68.1, C69.1, C74.1, C75.1, C76.1, C77.1, C82.1, C83.1, C84.1, C85.1, U10. (OUT), U11. (OUT), U12. (OUT), U13. (OUT), U14. (OUT), U15. (OUT), U16. (OUT), U17. (OUT), U18. (OUT), U19. (OUT), U20. (OUT), U21. (OUT), U22. (OUT), U23. (OUT), U24. (OUT), U25. (OUT), U26. (OUT), U27. (OUT), U28. (OUT), U29. (OUT), U31. (OUT), U32. (OUT), U33. (OUT), U34. (OUT), U35. (OUT), U36. (OUT), U37. (OUT), U5. (OUT), U6. (OUT), U7. (OUT), U8. (OUT), U9. (OUT)
- net HE0: now also U5.2 (OUT); no longer C33.2, C35.2, C37.2, C39.2, C43.2, C45.2, C47.2, C49.2, C50.2, C51.2, C53.2, C55.2, C57.2, C59.2, C60.2, C61.2, C66.2, C67.2, C68.2, C69.2, C74.2, C75.2, C76.2, C77.2, C82.2, C83.2, C84.2, C85.2, U10. (OUT), U11. (OUT), U12. (OUT), U13. (OUT), U14. (OUT), U15. (OUT), U16. (OUT), U17. (OUT), U18. (OUT), U19. (OUT), U20. (OUT), U21. (OUT), U22. (OUT), U23. (OUT), U24. (OUT), U25. (OUT), U26. (OUT), U27. (OUT), U28. (OUT), U29. (OUT), U31. (OUT), U32. (OUT), U33. (OUT), U34. (OUT), U35. (OUT), U36. (OUT), U37. (OUT), U6. (OUT), U9. (OUT)
- net HE1: now also C24.2, U6.2 (OUT); no longer C25.2, U5. (OUT)
- net HE10: now also C46.2, U17.2 (OUT)
- net HE11: now also C48.2, U18.2 (OUT)
- net HE12: now also C52.2, U20.2 (OUT)
- net HE13: now also C54.2, U21.2 (OUT)
- net HE14: now also C56.2, U22.2 (OUT)
- net HE15: now also C58.2, U23.2 (OUT)
- net HE16: now also C30.2, U9.2 (OUT)
- net HE17: now also C62.2, U25.2 (OUT)
- net HE18: now also C70.2, U29.2 (OUT)
- net HE19: now also C78.2, U34.2 (OUT)
- net HE2: now also C26.2, U7.2 (OUT); no longer C27.2, U7. (OUT)
- net HE20: now also C31.2, U14.2 (OUT)
- net HE21: now also C63.2, U26.2 (OUT)
- net HE22: now also C71.2, U31.2 (OUT)
- net HE23: now also C79.2, U35.2 (OUT)
- net HE24: now also C40.2, U19.2 (OUT)
- net HE25: now also C64.2, U27.2 (OUT)
- net HE26: now also C72.2, U32.2 (OUT)
- net HE27: now also C80.2, U36.2 (OUT)
- net HE28: now also C41.2, U24.2 (OUT)
- net HE29: now also C65.2, U28.2 (OUT)
- net HE3: now also C28.2, U8.2 (OUT); no longer C29.2, U8. (OUT)
- net HE30: now also C73.2, U33.2 (OUT)
- net HE31: now also C81.2, U37.2 (OUT)
- net HE4: now also C32.2, U10.2 (OUT)
- net HE5: now also C34.2, U11.2 (OUT)
- net HE6: now also C36.2, U12.2 (OUT)
- net HE7: now also C38.2, U13.2 (OUT)
- net HE8: now also C42.2, U15.2 (OUT)
- net HE9: now also C44.2, U16.2 (OUT)
- net LED: now also U1.13 (GPIO10), D1.3 (DIN); no longer U1.2 (GPIO0)
- net MUX_A_SEL0: now also U1.2 (GPIO0)
- net MUX_A_SEL1: now also U1.3 (GPIO1)
- net MUX_A_SEL2: now also U1.4 (GPIO2)
- net MUX_A_SEL3: now also U1.5 (GPIO3)
- net MUX_B_SEL0: now also U1.7 (GPIO5)
- net MUX_B_SEL1: now also U1.8 (GPIO6)
- net MUX_B_SEL2: now also U1.9 (GPIO7)
- net MUX_B_SEL3: now also U1.11 (GPIO8)
- net RESET: now also J3.1 (Pin_1)
- net SWC: now also J3.4 (Pin_4)
- net SWD: now also J3.5 (Pin_5)
- net MUX_A_OUT: now reaches U30.1 (COM)
- net MUX_A_OUT: now also U1.38 (GPIO26_ADC0)
- net MUX_B_OUT: now reaches U1.39 (GPIO27_ADC1)
- net MUX_B_OUT: now also U38.1 (COM)
- new net: D4.1 (DOUT), D5.3 (DIN)
- new net: D3.1 (DOUT), D4.3 (DIN)
- new net: D7.1 (DOUT), D8.3 (DIN)
- new net: D6.1 (DOUT), D7.3 (DIN)
- new net: D13.1 (DOUT), D14.3 (DIN)
- new net: D12.1 (DOUT), D13.3 (DIN)
- new net: D8.1 (DOUT), D9.3 (DIN)
- new net: D17.1 (DOUT), D18.3 (DIN)
- new net: D16.1 (DOUT), D17.3 (DIN)
- new net: D11.1 (DOUT), D12.3 (DIN)
- new net: D24.1 (DOUT), D25.3 (DIN)
- new net: D23.1 (DOUT), D24.3 (DIN)
- new net: D10.3 (DIN), D9.1 (DOUT)
- new net: D10.1 (DOUT), D5.1 (DOUT)
- new net: D18.1 (DOUT), D19.3 (DIN)
- new net: D15.1 (DOUT), D20.1 (DOUT)
- new net: D19.1 (DOUT), D20.3 (DIN)
- new net: D16.3 (DIN), D21.3 (DIN)
- new net: D1.1 (DOUT), D2.3 (DIN)
- new net: D22.1 (DOUT), D23.3 (DIN)
- new net: D14.1 (DOUT), D15.3 (DIN)
- new net: D2.1 (DOUT), D3.3 (DIN)
- new net: D21.1 (DOUT), D22.3 (DIN)
- new net: D11.3 (DIN), D6.3 (DIN)
- no-connect marks 5 -> 4
Other:
- moved on the sheet: C17, C18, C19, C20, C21, C22, C23, U30, U38

Commit message: finished schematic
Parts:
- removed C30, C31, C40, C41, C62, C63, C64, C65, C70, C71, C72, C73, C78, C79, C80, C81: 10pF, Capacitor_SMD:C_01005_0402Metric, symbol Device:C
- removed C50, C51, C60, C61, C66, C67, C68, C69, C74, C75, C76, C77, C82, C83, C84, C85: 1nF, Capacitor_SMD:C_01005_0402Metric, symbol Device:C
- removed J2: Conn_01x04, Connector_JST:JST_SH_SM04B-SRSS-TB_1x04-1MP_P1.00mm_Horizontal, symbol Connector_Generic:Conn_01x04
- removed U14, U19, U24, U25, U26, U27, U28, U29, U31, U32, U33, U34, U35, U36, U37, U9: ~, analog-keeb:HX6659-SOT23, symbol analog-keeb:HX6659
- removed U38: CD74HC4067SM, Package_SO:SSOP-24_5.3x8.2mm_P0.65mm, symbol 74xx:CD74HC4067SM
- added U14, U19, U24, U25, U26, U27, U28, U29, U31, U32, U33, U34, U35, U36, U37, U9: ~, lxsquid:Gateron_1.00u, symbol gateron-1.00u:gateron-1.00u
Connections:
- net HE0: now also C32.2, C42.2, C52.2, U10.2 (OUT), U15.2 (OUT), U20.2 (OUT)
- net HE1: now also C34.2, C44.2, C54.2, U11.2 (OUT), U16.2 (OUT), U21.2 (OUT)
- net HE10: no longer C46.2, U17.2 (OUT)
- net HE11: no longer C48.2, U18.2 (OUT)
- net HE12: no longer C52.2, U20.2 (OUT)
- net HE13: no longer C54.2, U21.2 (OUT)
- net HE14: no longer C56.2, U22.2 (OUT)
- net HE15: no longer C58.2, U23.2 (OUT)
- net HE2: now also C36.2, C46.2, C56.2, U12.2 (OUT), U17.2 (OUT), U22.2 (OUT)
- net HE3: now also C38.2, C48.2, C58.2, U13.2 (OUT), U18.2 (OUT), U23.2 (OUT)
- net HE4: no longer C32.2, U10.2 (OUT)
- net HE5: no longer C34.2, U11.2 (OUT)
- net HE6: no longer C36.2, U12.2 (OUT)
- net HE7: no longer C38.2, U13.2 (OUT)
- net HE8: no longer C42.2, U15.2 (OUT)
- net HE9: no longer C44.2, U16.2 (OUT)
- net LED: now also D25.1 (DOUT)
- net MUX_B_OUT: no longer names the net of U1.39 (GPIO27_ADC1)
- net MUX_B_SEL0: no longer names the net of U1.7 (GPIO5)
- net MUX_B_SEL1: no longer names the net of U1.8 (GPIO6)
- net MUX_B_SEL2: no longer names the net of U1.9 (GPIO7)
- net MUX_B_SEL3: no longer names the net of U1.11 (GPIO8)
Other:
- note added: "MUX1"
- moved on the sheet: C100, C101, C102, C103, C104, C105, C17, C18, C19, C20, C21, C86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

Commit message: trol
Connections:
- net +5V: now also U30.24 (VCC)
- net D+: now also U3.4 (IO3); no longer U3.1 (IO1)
Changed lines of the file:
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@@
 	)
 	(no_connect
-		(at 195.58 64.77)
+		(at 60.96 77.47)
 	)
 	(no_connect
-		(at 60.96 77.47)
+		(at 195.58 64.77)
 	)
 	(no_connect
-		(at 60.96 74.93)
+		(at 170.18 59.69)
 	)
 	(no_connect
-		(at 195.58 59.69)
+		(at 60.96 74.93)
 	)
 	(wire
@@
 	(wire
 		(pts
+			(xy 182.88 138.43) (xy 182.88 143.51)
+		)
+		(stroke
+			(width 0)
+			(type default)
+		)
+	)
+	(wire
+		(pts
 			(xy 405.13 125.73) (xy 405.13 137.16)
 		)
@@
 	(global_label "D+"
 		(shape input)
-		(at 170.18 59.69 180)
+		(at 195.58 59.69 0)
 		(fields_autoplaced yes)
 		(effects
@@
 				(size 1.27 1.27)
 			)
-			(justify right)
+			(justify left)
 		)
 		(property "Intersheetrefs" "${INTERSHEET_REFS}"
-			(at 164.3524 59.69 0)
+			(at 201.4076 59.69 0)
 			(effects
 				(font
 					(size 1.27 1.27)
 				)
-				(justify right)
+				(justify left)
 				(hide yes)
 			)
@@
 					(unit 1)
 				)
+			)
+		)
+	)
+	(symbol
+		(lib_id "power:+5V")
+		(at 182.88 138.43 0)
+		(unit 1)
+		(exclude_from_sim no)
+		(in_bom yes)
+		(on_board yes)
+		(dnp no)
+		(fields_autoplaced yes)
+		(property "Reference" "#PWR042"
+			(at 182.88 142.24 0)
+			(effects
+				(font
+					(size 1.27 1.27)
+				)
+				(hide yes)
+			)
+		)
+		(property "Value" "+5V"
+			(at 182.88 133.35 0)
+			(effects
+				(font
+					(size 1.27 1.27)
+				)
+			)
+		)
+		(property "Footprint" ""
+			(at 182.88 138.43 0)
+			(effects
+				(font
+					(size 1.27 1.27)
+				)
+				(hide yes)
+			)
+		)
+		(property "Datasheet" ""
+			(at 182.88 138.43 0)
+			(effects
+				(font
+					(size 1.27 1.27)
+				)
+				(hide yes)
+			)
+		)
+		(property "Description" "Power symbol creates a global label with name \"+5V\""
+			(at 182.88 138.43 0)
+			(effects
+				(font
+					(size 1.27 1.27)
+				)
+				(hide yes)
+			)
+		)
+		(pin "1"
+		)
+		(instances
+			(project "analog-keeb-proto"
+				(path "/0f7d2ff7-19be-4cc1-8cf4-df7d811021d2"
+					(reference "#PWR042")
+					(unit 1)
+				)
